Commit message: Update the other dual-arm URDFs to match the correct orientation of the arms

File: husky_ur_description/urdf/husky_dual_ur3_description.urdf.xacro (robot description, xacro)
@@ -16,4 +16,16 @@
     </collision>
   </link>
+  <link name="left_arm_bulkhead_link" />
+  <joint name="left_arm_bulkhead_joint" type="fixed">
+    <parent link="dual_arm_bulkhead_link" />
+    <child link="left_arm_bulkhead_link" />
+    <origin xyz="0.1225 0.14891 0.13371" rpy="0 -${pi/4} -${pi/2}"/>
+  </joint>
+  <link name="right_arm_bulkhead_link" />
+  <joint name="right_arm_bulkhead_joint" type="fixed">
+    <parent link="dual_arm_bulkhead_link" />
+    <child link="right_arm_bulkhead_link" />
+    <origin xyz="0.1225 -0.14891 0.13371" rpy="0 ${pi/4} -${pi/2}"/>
+  </joint>
   <joint name="dual_arm_bulkhead_joint" type="fixed">
     <parent link="base_link"/>
@@ -22,12 +34,12 @@
   </joint>
   <joint name="left_arm_mount_joint" type="fixed">
-    <parent link="dual_arm_bulkhead_link" />
+    <parent link="left_arm_bulkhead_link" />
     <child link="left_ur_arm_base_link" />
-    <origin xyz="$(optenv HUSKY_LEFT_UR_XYZ 0.1225 0.14891 0.13371)" rpy="$(optenv HUSKY_LEFT_UR_RPY 0.785398 0 3.14159)"/>
+    <origin xyz="$(optenv HUSKY_LEFT_UR_XYZ 0 0 0)" rpy="$(optenv HUSKY_LEFT_UR_RPY 0 0 0)"/>
   </joint>
   <joint name="right_arm_mount_joint" type="fixed">
-    <parent link="dual_arm_bulkhead_link" />
+    <parent link="right_arm_bulkhead_link" />
     <child link="right_ur_arm_base_link" />
-    <origin xyz="$(optenv HUSKY_RIGHT_UR_XYZ 0.1225 -0.14891 0.13371)" rpy="$(optenv HUSKY_RIGHT_UR_RPY 0.785398 0 0)"/>
+    <origin xyz="$(optenv HUSKY_RIGHT_UR_XYZ 0 0 0)" rpy="$(optenv HUSKY_RIGHT_UR_RPY 0 0 0)"/>
   </joint>
   <xacro:ur3_robot prefix="right_ur_arm_" />

File: husky_ur_description/urdf/husky_dual_ur3_e_description.urdf.xacro (robot description, xacro)
@@ -16,4 +16,16 @@
     </collision>
   </link>
+  <link name="left_arm_bulkhead_link" />
+  <joint name="left_arm_bulkhead_joint" type="fixed">
+    <parent link="dual_arm_bulkhead_link" />
+    <child link="left_arm_bulkhead_link" />
+    <origin xyz="0.1225 0.14891 0.13371" rpy="0 -${pi/4} -${pi/2}"/>
+  </joint>
+  <link name="right_arm_bulkhead_link" />
+  <joint name="right_arm_bulkhead_joint" type="fixed">
+    <parent link="dual_arm_bulkhead_link" />
+    <child link="right_arm_bulkhead_link" />
+    <origin xyz="0.1225 -0.14891 0.13371" rpy="0 ${pi/4} -${pi/2}"/>
+  </joint>
   <joint name="dual_arm_bulkhead_joint" type="fixed">
     <parent link="base_link"/>
@@ -22,12 +34,12 @@
   </joint>
   <joint name="left_arm_mount_joint" type="fixed">
-    <parent link="dual_arm_bulkhead_link" />
+    <parent link="left_arm_bulkhead_link" />
     <child link="left_ur_arm_base_link" />
-    <origin xyz="$(optenv HUSKY_LEFT_UR_XYZ 0.1225 0.14891 0.13371)" rpy="$(optenv HUSKY_LEFT_UR_RPY 0.785398 0 3.14159)"/>
+    <origin xyz="$(optenv HUSKY_LEFT_UR_XYZ 0 0 0)" rpy="$(optenv HUSKY_LEFT_UR_RPY 0 0 0)"/>
   </joint>
   <joint name="right_arm_mount_joint" type="fixed">
-    <parent link="dual_arm_bulkhead_link" />
+    <parent link="right_arm_bulkhead_link" />
     <child link="right_ur_arm_base_link" />
-    <origin xyz="$(optenv HUSKY_RIGHT_UR_XYZ 0.1225 -0.14891 0.13371)" rpy="$(optenv HUSKY_RIGHT_UR_RPY 0.785398 0 0)"/>
+    <origin xyz="$(optenv HUSKY_RIGHT_UR_XYZ 0 0 0)" rpy="$(optenv HUSKY_RIGHT_UR_RPY 0 0 0)"/>
   </joint>
   <xacro:ur3e_robot prefix="right_ur_arm_" />

File: husky_ur_description/urdf/husky_dual_ur5_description.urdf.xacro (robot description, xacro)
@@ -16,4 +16,16 @@
     </collision>
   </link>
+  <link name="left_arm_bulkhead_link" />
+  <joint name="left_arm_bulkhead_joint" type="fixed">
+    <parent link="dual_arm_bulkhead_link" />
+    <child link="left_arm_bulkhead_link" />
+    <origin xyz="0.1225 0.14891 0.13371" rpy="0 -${pi/4} -${pi/2}"/>
+  </joint>
+  <link name="right_arm_bulkhead_link" />
+  <joint name="right_arm_bulkhead_joint" type="fixed">
+    <parent link="dual_arm_bulkhead_link" />
+    <child link="right_arm_bulkhead_link" />
+    <origin xyz="0.1225 -0.14891 0.13371" rpy="0 ${pi/4} -${pi/2}"/>
+  </joint>
   <joint name="dual_arm_bulkhead_joint" type="fixed">
     <parent link="base_link"/>
@@ -22,12 +34,12 @@
   </joint>
   <joint name="left_arm_mount_joint" type="fixed">
-    <parent link="dual_arm_bulkhead_link" />
+    <parent link="left_arm_bulkhead_link" />
     <child link="left_ur_arm_base_link" />
-    <origin xyz="$(optenv HUSKY_LEFT_UR_XYZ 0.1225 0.14891 0.13371)" rpy="$(optenv HUSKY_LEFT_UR_RPY 0.785398 0 3.14159)"/>
+    <origin xyz="$(optenv HUSKY_LEFT_UR_XYZ 0 0 0)" rpy="$(optenv HUSKY_LEFT_UR_RPY 0 0 0)"/>
   </joint>
   <joint name="right_arm_mount_joint" type="fixed">
-    <parent link="dual_arm_bulkhead_link" />
+    <parent link="right_arm_bulkhead_link" />
     <child link="right_ur_arm_base_link" />
-    <origin xyz="$(optenv HUSKY_RIGHT_UR_XYZ 0.1225 -0.14891 0.13371)" rpy="$(optenv HUSKY_RIGHT_UR_RPY 0.785398 0 0)"/>
+    <origin xyz="$(optenv HUSKY_RIGHT_UR_XYZ 0 0 0)" rpy="$(optenv HUSKY_RIGHT_UR_RPY 0 0 0)"/>
   </joint>
   <xacro:ur5_robot prefix="right_ur_arm_" />

Commit message: Added robotiq as argument and environemnt var to URDF

File: husky_ur_description/urdf/husky_dual_ur3_description.urdf.xacro (robot description, xacro)
@@ -2,4 +2,12 @@
 <robot xmlns:xacro="http://ros.org/wiki/xacro">
   <xacro:include filename="$(find ur_description)/urdf/inc/ur3_macro.xacro" />
+  <!-- Parameters -->
+  <xacro:arg name="left_arm_xyz"  default="$(optenv HUSKY_LEFT_UR_XYZ 0.1225 0.14891 0.13371)" />
+  <xacro:arg name="left_arm_rpy"  default="$(optenv HUSKY_LEFT_UR_RPY 0.785398 0 3.14159)" />
+  <xacro:arg name="right_arm_xyz" default="$(optenv HUSKY_RIGHT_UR_XYZ 0.1225 -0.14891 0.13371)" />
+  <xacro:arg name="right_arm_rpy" default="$(optenv HUSKY_RIGHT_UR_RPY 0.785398 0 0)" />
+  <xacro:arg name="left_arm_gripper_enable" default="$(optenv HUSKY_LEFT_UR_GRIPPER_ENABLED 0)" />
+  <xacro:arg name="right_arm_gripper_enable" default="$(optenv HUSKY_RIGHT_UR_GRIPPER_ENABLED 0)" />
+  <!-- Bulk Head -->
   <link name="dual_arm_bulkhead_link">
     <visual>
@@ -24,12 +32,22 @@
     <parent link="dual_arm_bulkhead_link" />
     <child link="left_ur_arm_base_link" />
-    <origin xyz="$(optenv HUSKY_LEFT_UR_XYZ 0.1225 0.14891 0.13371)" rpy="$(optenv HUSKY_LEFT_UR_RPY 0.785398 0 3.14159)"/>
+    <origin xyz="$(arg left_arm_xyz)" rpy="$(arg left_arm_rpy)"/>
   </joint>
   <joint name="right_arm_mount_joint" type="fixed">
     <parent link="dual_arm_bulkhead_link" />
     <child link="right_ur_arm_base_link" />
-    <origin xyz="$(optenv HUSKY_RIGHT_UR_XYZ 0.1225 -0.14891 0.13371)" rpy="$(optenv HUSKY_RIGHT_UR_RPY 0.785398 0 0)"/>
+    <origin xyz="$(arg right_arm_xyz)" rpy="$(arg right_arm_rpy)"/>
   </joint>
+  <!-- Arms -->
   <xacro:ur3_robot prefix="right_ur_arm_" />
   <xacro:ur3_robot prefix="left_ur_arm_" />
+  <!-- Grippers -->
+  <xacro:if value="$(arg left_arm_gripper_enable)">
+    <xacro:include filename="$(find husky_ur_description)/urdf/inc/ur_robotiq_2f_gripper.urdf.xacro" />
+    <xacro:ur_robotiq_2f_gripper prefix="left_ur_arm_gripper" parent="left_ur_arm_tool0" />
+  </xacro:if>
+  <xacro:if value="$(arg right_arm_gripper_enable)">
+    <xacro:include filename="$(find husky_ur_description)/urdf/inc/ur_robotiq_2f_gripper.urdf.xacro" />
+    <xacro:ur_robotiq_2f_gripper prefix="right_ur_arm_gripper" parent="right_ur_arm_tool0" />
+  </xacro:if>
 </robot>

File: husky_ur_description/urdf/husky_dual_ur3_e_description.urdf.xacro (robot description, xacro)
@@ -2,4 +2,12 @@
 <robot xmlns:xacro="http://ros.org/wiki/xacro">
   <xacro:include filename="$(find ur_description)/urdf/inc/ur3e_macro.xacro" />
+  <!-- Parameters -->
+  <xacro:arg name="left_arm_xyz"  default="$(optenv HUSKY_LEFT_UR_XYZ 0.1225 0.14891 0.13371)" />
+  <xacro:arg name="left_arm_rpy"  default="$(optenv HUSKY_LEFT_UR_RPY 0.785398 0 3.14159)" />
+  <xacro:arg name="right_arm_xyz" default="$(optenv HUSKY_RIGHT_UR_XYZ 0.1225 -0.14891 0.13371)" />
+  <xacro:arg name="right_arm_rpy" default="$(optenv HUSKY_RIGHT_UR_RPY 0.785398 0 0)" />
+  <xacro:arg name="left_arm_gripper_enable" default="$(optenv HUSKY_LEFT_UR_GRIPPER_ENABLED 0)" />
+  <xacro:arg name="right_arm_gripper_enable" default="$(optenv HUSKY_RIGHT_UR_GRIPPER_ENABLED 0)" />
+  <!-- Bulk Head -->
   <link name="dual_arm_bulkhead_link">
     <visual>
@@ -24,12 +32,22 @@
     <parent link="dual_arm_bulkhead_link" />
     <child link="left_ur_arm_base_link" />
-    <origin xyz="$(optenv HUSKY_LEFT_UR_XYZ 0.1225 0.14891 0.13371)" rpy="$(optenv HUSKY_LEFT_UR_RPY 0.785398 0 3.14159)"/>
+    <origin xyz="$(arg left_arm_xyz)" rpy="$(arg left_arm_rpy)"/>
   </joint>
   <joint name="right_arm_mount_joint" type="fixed">
     <parent link="dual_arm_bulkhead_link" />
     <child link="right_ur_arm_base_link" />
-    <origin xyz="$(optenv HUSKY_RIGHT_UR_XYZ 0.1225 -0.14891 0.13371)" rpy="$(optenv HUSKY_RIGHT_UR_RPY 0.785398 0 0)"/>
+    <origin xyz="$(arg right_arm_xyz)" rpy="$(arg right_arm_rpy)"/>
   </joint>
+  <!-- Arms -->
   <xacro:ur3e_robot prefix="right_ur_arm_" />
   <xacro:ur3e_robot prefix="left_ur_arm_" />
+  <!-- Grippers -->
+  <xacro:if value="$(arg left_arm_gripper_enable)">
+    <xacro:include filename="$(find husky_ur_description)/urdf/inc/ur_robotiq_2f_gripper.urdf.xacro" />
+    <xacro:ur_robotiq_2f_gripper prefix="left_ur_arm_gripper" parent="left_ur_arm_tool0" />
+  </xacro:if>
+  <xacro:if value="$(arg right_arm_gripper_enable)">
+    <xacro:include filename="$(find husky_ur_description)/urdf/inc/ur_robotiq_2f_gripper.urdf.xacro" />
+    <xacro:ur_robotiq_2f_gripper prefix="right_ur_arm_gripper" parent="right_ur_arm_tool0" />
+  </xacro:if>
 </robot>

File: husky_ur_description/urdf/husky_dual_ur5_description.urdf.xacro (robot description, xacro)
@@ -2,4 +2,12 @@
 <robot xmlns:xacro="http://ros.org/wiki/xacro">
   <xacro:include filename="$(find ur_description)/urdf/inc/ur5_macro.xacro" />
+  <!-- Parameters -->
+  <xacro:arg name="left_arm_xyz"  default="$(optenv HUSKY_LEFT_UR_XYZ 0.1225 0.14891 0.13371)" />
+  <xacro:arg name="left_arm_rpy"  default="$(optenv HUSKY_LEFT_UR_RPY 0.785398 0 3.14159)" />
+  <xacro:arg name="right_arm_xyz" default="$(optenv HUSKY_RIGHT_UR_XYZ 0.1225 -0.14891 0.13371)" />
+  <xacro:arg name="right_arm_rpy" default="$(optenv HUSKY_RIGHT_UR_RPY 0.785398 0 0)" />
+  <xacro:arg name="left_arm_gripper_enable" default="$(optenv HUSKY_LEFT_UR_GRIPPER_ENABLED 0)" />
+  <xacro:arg name="right_arm_gripper_enable" default="$(optenv HUSKY_RIGHT_UR_GRIPPER_ENABLED 0)" />
+  <!-- Bulk Head -->
   <link name="dual_arm_bulkhead_link">
     <visual>
@@ -24,12 +32,22 @@
     <parent link="dual_arm_bulkhead_link" />
     <child link="left_ur_arm_base_link" />
-    <origin xyz="$(optenv HUSKY_LEFT_UR_XYZ 0.1225 0.14891 0.13371)" rpy="$(optenv HUSKY_LEFT_UR_RPY 0.785398 0 3.14159)"/>
+    <origin xyz="$(arg left_arm_xyz)" rpy="$(arg left_arm_rpy)"/>
   </joint>
   <joint name="right_arm_mount_joint" type="fixed">
     <parent link="dual_arm_bulkhead_link" />
     <child link="right_ur_arm_base_link" />
-    <origin xyz="$(optenv HUSKY_RIGHT_UR_XYZ 0.1225 -0.14891 0.13371)" rpy="$(optenv HUSKY_RIGHT_UR_RPY 0.785398 0 0)"/>
+    <origin xyz="$(arg right_arm_xyz)" rpy="$(arg right_arm_rpy)"/>
   </joint>
+  <!-- Arms -->
   <xacro:ur5_robot prefix="right_ur_arm_" />
   <xacro:ur5_robot prefix="left_ur_arm_" />
+  <!-- Grippers -->
+  <xacro:if value="$(arg left_arm_gripper_enable)">
+    <xacro:include filename="$(find husky_ur_description)/urdf/inc/ur_robotiq_2f_gripper.urdf.xacro" />
+    <xacro:ur_robotiq_2f_gripper prefix="left_ur_arm_gripper" parent="left_ur_arm_tool0" />
+  </xacro:if>
+  <xacro:if value="$(arg right_arm_gripper_enable)">
+    <xacro:include filename="$(find husky_ur_description)/urdf/inc/ur_robotiq_2f_gripper.urdf.xacro" />
+    <xacro:ur_robotiq_2f_gripper prefix="right_ur_arm_gripper" parent="right_ur_arm_tool0" />
+  </xacro:if>
 </robot>

File: husky_ur_description/urdf/husky_dual_ur5_e_description.urdf.xacro (robot description, xacro)
@@ -2,4 +2,12 @@
 <robot xmlns:xacro="http://ros.org/wiki/xacro">
   <xacro:include filename="$(find ur_description)/urdf/inc/ur5e_macro.xacro" />
+  <!-- Parameters -->
+  <xacro:arg name="left_arm_xyz"  default="$(optenv HUSKY_LEFT_UR_XYZ 0.1225 0.14891 0.13371)" />
+  <xacro:arg name="left_arm_rpy"  default="$(optenv HUSKY_LEFT_UR_RPY 0.785398 0 3.14159)" />
+  <xacro:arg name="right_arm_xyz" default="$(optenv HUSKY_RIGHT_UR_XYZ 0.1225 -0.14891 0.13371)" />
+  <xacro:arg name="right_arm_rpy" default="$(optenv HUSKY_RIGHT_UR_RPY 0.785398 0 0)" />
+  <xacro:arg name="left_arm_gripper_enable" default="$(optenv HUSKY_LEFT_UR_GRIPPER_ENABLED 0)" />
+  <xacro:arg name="right_arm_gripper_enable" default="$(optenv HUSKY_RIGHT_UR_GRIPPER_ENABLED 0)" />
+  <!-- Bulk Head -->
   <link name="dual_arm_bulkhead_link">
     <visual>
@@ -24,12 +32,22 @@
     <parent link="dual_arm_bulkhead_link" />
     <child link="left_ur_arm_base_link" />
-    <origin xyz="$(optenv HUSKY_LEFT_UR_XYZ 0.1225 0.14891 0.13371)" rpy="$(optenv HUSKY_LEFT_UR_RPY 0.785398 0 3.14159)"/>
+    <origin xyz="$(arg left_arm_xyz)" rpy="$(arg left_arm_rpy)"/>
   </joint>
   <joint name="right_arm_mount_joint" type="fixed">
     <parent link="dual_arm_bulkhead_link" />
     <child link="right_ur_arm_base_link" />
-    <origin xyz="$(optenv HUSKY_RIGHT_UR_XYZ 0.1225 -0.14891 0.13371)" rpy="$(optenv HUSKY_RIGHT_UR_RPY 0.785398 0 0)"/>
+    <origin xyz="$(arg right_arm_xyz)" rpy="$(arg right_arm_rpy)"/>
   </joint>
+  <!-- Arms -->
   <xacro:ur5e_robot prefix="right_ur_arm_" />
   <xacro:ur5e_robot prefix="left_ur_arm_" />
+  <!-- Grippers -->
+  <xacro:if value="$(arg left_arm_gripper_enable)">
+    <xacro:include filename="$(find husky_ur_description)/urdf/inc/ur_robotiq_2f_gripper.urdf.xacro" />
+    <xacro:ur_robotiq_2f_gripper prefix="left_ur_arm_gripper" parent="left_ur_arm_tool0" />
+  </xacro:if>
+  <xacro:if value="$(arg right_arm_gripper_enable)">
+    <xacro:include filename="$(find husky_ur_description)/urdf/inc/ur_robotiq_2f_gripper.urdf.xacro" />
+    <xacro:ur_robotiq_2f_gripper prefix="right_ur_arm_gripper" parent="right_ur_arm_tool0" />
+  </xacro:if>
 </robot>

File: husky_ur_description/urdf/husky_ur3_description.urdf.xacro (robot description, xacro)
@@ -2,9 +2,18 @@
 <robot xmlns:xacro="http://ros.org/wiki/xacro">
   <xacro:include filename="$(find ur_description)/urdf/inc/ur3_macro.xacro" />
+  <!-- Parameters -->
+  <xacro:arg name="arm_xyz" default="$(optenv HUSKY_UR_XYZ -0.105 0.0 0.0)"/>
+  <xacro:arg name="arm_rpy" default="$(optenv HUSKY_UR_RPY 0 0 3.1415927)"/>
+  <xacro:arg name="arm_gripper_enable" default="$(optenv HUSKY_UR_GRIPPER_ENABLED 0)" />
   <joint name="arm_mount_joint" type="fixed">
     <parent link="top_plate_front_link" />
     <child link="ur_arm_base_link" />
-    <origin xyz="$(optenv HUSKY_UR_XYZ -0.105 0.0 0.0)" rpy="$(optenv HUSKY_UR_RPY 0 0 3.1415927)"/>
+    <origin xyz="$(arg arm_xyz)" rpy="$(arg arm_rpy)"/>
   </joint>
   <xacro:ur3_robot prefix="ur_arm_" />
+  <!-- Grippers -->
+  <xacro:if value="$(arg arm_gripper_enable)">
+    <xacro:include filename="$(find husky_ur_description)/urdf/inc/ur_robotiq_2f_gripper.urdf.xacro" />
+    <xacro:ur_robotiq_2f_gripper prefix="ur_arm_gripper" parent="ur_arm_tool0" />
+  </xacro:if>
 </robot>

File: husky_ur_description/urdf/husky_ur3_e_description.urdf.xacro (robot description, xacro)
@@ -2,9 +2,18 @@
 <robot xmlns:xacro="http://ros.org/wiki/xacro">
   <xacro:include filename="$(find ur_description)/urdf/inc/ur3e_macro.xacro" />
+  <!-- Parameters -->
+  <xacro:arg name="arm_xyz" default="$(optenv HUSKY_UR_XYZ -0.105 0.0 0.0)"/>
+  <xacro:arg name="arm_rpy" default="$(optenv HUSKY_UR_RPY 0 0 3.1415927)"/>
+  <xacro:arg name="arm_gripper_enable" default="$(optenv HUSKY_UR_GRIPPER_ENABLED 0)" />
   <joint name="arm_mount_joint" type="fixed">
     <parent link="top_plate_front_link" />
     <child link="ur_arm_base_link" />
-    <origin xyz="$(optenv HUSKY_UR_XYZ -0.105 0.0 0.0)" rpy="$(optenv HUSKY_UR_RPY 0 0 3.1415927)"/>
+    <origin xyz="$(arg arm_xyz)" rpy="$(arg arm_rpy)"/>
   </joint>
   <xacro:ur3e_robot prefix="ur_arm_" />
+  <!-- Grippers -->
+  <xacro:if value="$(arg arm_gripper_enable)">
+    <xacro:include filename="$(find husky_ur_description)/urdf/inc/ur_robotiq_2f_gripper.urdf.xacro" />
+    <xacro:ur_robotiq_2f_gripper prefix="ur_arm_gripper" parent="ur_arm_tool0" />
+  </xacro:if>
 </robot>

File: husky_ur_description/urdf/husky_ur5_description.urdf.xacro (robot description, xacro)
@@ -2,9 +2,18 @@
 <robot xmlns:xacro="http://ros.org/wiki/xacro">
   <xacro:include filename="$(find ur_description)/urdf/inc/ur5_macro.xacro" />
+  <!-- Parameters -->
+  <xacro:arg name="arm_xyz" default="$(optenv HUSKY_UR_XYZ -0.105 0.0 0.0)"/>
+  <xacro:arg name="arm_rpy" default="$(optenv HUSKY_UR_RPY 0 0 3.1415927)"/>
+  <xacro:arg name="arm_gripper_enable" default="$(optenv HUSKY_UR_GRIPPER_ENABLED 0)" />
   <joint name="arm_mount_joint" type="fixed">
     <parent link="top_plate_front_link" />
     <child link="ur_arm_base_link" />
-    <origin xyz="$(optenv HUSKY_UR_XYZ -0.105 0.0 0.0)" rpy="$(optenv HUSKY_UR_RPY 0 0 3.1415927)"/>
+    <origin xyz="$(arg arm_xyz)" rpy="$(arg arm_rpy)"/>
   </joint>
   <xacro:ur5_robot prefix="ur_arm_" />
+  <!-- Grippers -->
+  <xacro:if value="$(arg arm_gripper_enable)">
+    <xacro:include filename="$(find husky_ur_description)/urdf/inc/ur_robotiq_2f_gripper.urdf.xacro" />
+    <xacro:ur_robotiq_2f_gripper prefix="ur_arm_gripper" parent="ur_arm_tool0" />
+  </xacro:if>
 </robot>

File: husky_ur_description/urdf/husky_ur5_e_description.urdf.xacro (robot description, xacro)
@@ -2,9 +2,18 @@
 <robot xmlns:xacro="http://ros.org/wiki/xacro">
   <xacro:include filename="$(find ur_description)/urdf/inc/ur5e_macro.xacro" />
+  <!-- Parameters -->
+  <xacro:arg name="arm_xyz" default="$(optenv HUSKY_UR_XYZ -0.105 0.0 0.0)"/>
+  <xacro:arg name="arm_rpy" default="$(optenv HUSKY_UR_RPY 0 0 3.1415927)"/>
+  <xacro:arg name="arm_gripper_enable" default="$(optenv HUSKY_UR_GRIPPER_ENABLED 0)" />
   <joint name="arm_mount_joint" type="fixed">
     <parent link="top_plate_front_link" />
     <child link="ur_arm_base_link" />
-    <origin xyz="$(optenv HUSKY_UR_XYZ -0.105 0.0 0.0)" rpy="$(optenv HUSKY_UR_RPY 0 0 3.1415927)"/>
+    <origin xyz="$(arg arm_xyz)" rpy="$(arg arm_rpy)"/>
   </joint>
   <xacro:ur5e_robot prefix="ur_arm_" />
+  <!-- Grippers -->
+  <xacro:if value="$(arg arm_gripper_enable)">
+    <xacro:include filename="$(find husky_ur_description)/urdf/inc/ur_robotiq_2f_gripper.urdf.xacro" />
+    <xacro:ur_robotiq_2f_gripper prefix="ur_arm_gripper" parent="ur_arm_tool0" />
+  </xacro:if>
 </robot>
