Commit message: Updated gen3 descriptions

File: husky_kinova_description/urdf/husky_gen3_robotiq_2f_140_description.urdf.xacro (robot description, xacro)
@@ -4,5 +4,5 @@
   <xacro:arg name="dof" default="7" />
   <xacro:arg name="vision" default="true" />
-  <xacro:arg name="gripper" default="" />
+  <xacro:arg name="gripper" default="robotiq_2f_140" />
   <xacro:arg name="sim" default="false" />
   <xacro:arg name="prefix" default="kinova_arm_" />

File: husky_kinova_description/urdf/husky_gen3_robotiq_2f_85_description.urdf.xacro (robot description, xacro)
@@ -1,9 +1,16 @@
 <?xml version="1.0"?>
 <robot xmlns:xacro="http://ros.org/wiki/xacro">
-  <xacro:include filename="$(find kortex_description)/robots/gen3_robotiq_2f_85.xacro" />
+  <xacro:arg name="arm" default="gen3" />
+  <xacro:arg name="dof" default="7" />
+  <xacro:arg name="vision" default="true" />
+  <xacro:arg name="gripper" default="robotiq_2f_85" />
+  <xacro:arg name="sim" default="false" />
+  <xacro:arg name="prefix" default="kinova_arm_" />
+  <xacro:include filename="$(find kortex_description)/robots/kortex_robot.xacro" />
+  <xacro:load_robot arm="$(arg arm)" gripper="$(arg gripper)" dof="$(arg dof)" vision="$(arg vision)" sim="$(arg sim)" prefix="$(arg prefix)" />
   <joint name="arm_mount_joint" type="fixed">
-    <origin xyz="$(optenv HUSKY_KINOVA_XYZ -0.105 0 0)" rpy="$(optenv HUSKY_KINOVA_RPY 0 0 0)" />
+    <origin xyz="$(optenv HUSKY_KINOVA_XYZ -0.105 0.0 0.0)" rpy="$(optenv HUSKY_KINOVA_RPY 0 0 0)" />
     <parent link="top_plate_front_link" />
-    <child link="arm_base_link" />
+    <child link="kinova_arm_base_link" />
   </joint>
 </robot>
