Commit message: Initial pass at franka bringup and moveit.  All I can do until I get to a real arm

File: husky_franka_description/urdf/husky_panda_hand_description.urdf.xacro (robot description, xacro)
@@ -4,5 +4,5 @@
     <parent link="base_link" />
     <child link="franka_mount_link" />
-    <origin xyz="$(optenv HUSKY_FRANKA_XYZ 0.494 0 0.225)" rpy="$(optenv HUSKY_FRANKA_RPY 0 0 0)"/>
+    <origin xyz="$(optenv HUSKY_FRANKA_XYZ 0.375 0 0.234)" rpy="$(optenv HUSKY_FRANKA_RPY 0 0 0)"/>
   </joint>
   <link name="franka_mount_link" />
