Commit message: Added Reference Pose

File: husky_franka_moveit_config/config/arm.xacro (robot description, xacro)
@@ -11,20 +11,29 @@
         </group>
         <!--GROUP STATES: Purpose: Define a named state for a particular group, in terms of joint values. This is useful to define states like 'folded arms'-->
-        <group_state name="ready" group="${name}">
-            <joint name="$(arg arm_id)_joint1" value="0" />
-            <joint name="$(arg arm_id)_joint2" value="${-pi/4}" />
-            <joint name="$(arg arm_id)_joint3" value="0" />
-            <joint name="$(arg arm_id)_joint4" value="${-3*pi/4}" />
-            <joint name="$(arg arm_id)_joint5" value="0" />
-            <joint name="$(arg arm_id)_joint6" value="${pi/2}" />
-            <joint name="$(arg arm_id)_joint7" value="${pi/4}" />
-        </group_state>
-        <group_state name="extended" group="${name}">
+        <group_state name="reference" group="${name}">
             <joint name="$(arg arm_id)_joint1" value="0" />
             <joint name="$(arg arm_id)_joint2" value="0" />
             <joint name="$(arg arm_id)_joint3" value="0" />
-            <joint name="$(arg arm_id)_joint4" value="-0.1" />
+            <joint name="$(arg arm_id)_joint4" value="${-pi/2}" />
+            <joint name="$(arg arm_id)_joint5" value="0" />
+            <joint name="$(arg arm_id)_joint6" value="${pi/2}" />
+            <joint name="$(arg arm_id)_joint7" value="0" />
+        </group_state>
+        <group_state name="ready" group="${name}">
+            <joint name="$(arg arm_id)_joint1" value="0" />
+            <joint name="$(arg arm_id)_joint2" value="0" />
+            <joint name="$(arg arm_id)_joint3" value="0" />
+            <joint name="$(arg arm_id)_joint4" value="${-pi/2}" />
             <joint name="$(arg arm_id)_joint5" value="0" />
             <joint name="$(arg arm_id)_joint6" value="${pi}" />
+            <joint name="$(arg arm_id)_joint7" value="${pi/4}" />
+        </group_state>
+        <group_state name="all_zeros" group="${name}">
+            <joint name="$(arg arm_id)_joint1" value="0" />
+            <joint name="$(arg arm_id)_joint2" value="0" />
+            <joint name="$(arg arm_id)_joint3" value="0" />
+            <joint name="$(arg arm_id)_joint4" value="0" />
+            <joint name="$(arg arm_id)_joint5" value="0" />
+            <joint name="$(arg arm_id)_joint6" value="0" />
             <joint name="$(arg arm_id)_joint7" value="${pi/4}" />
         </group_state>
